File: rc-debouncer/rc-debouncer.kicad_pcb (KiCad board)
At the start: 2 copper layers, 26 parts, among them J1 MCU, J2 SIG.IN, SW1 Input, U1 LM311

Commit message: Finish layout and generate production outputs
Parts:
- added C7: 100nF, Capacitor_THT:C_Disc_D3.0mm_W2.0mm_P2.50mm, F.Cu at (237.5, 113.0)
- added REF**: OSHW-Logo_7.5x8mm_SilkScreen, Symbol:OSHW-Logo_7.5x8mm_SilkScreen, B.Cu at (203.8, 88.3)
- added U2: LM358, Package_DIP:DIP-8_W7.62mm_LongPads, F.Cu at (233.7, 105.4)
- J1: footprint Connector_JST:JST_XH_B3B-XH-A_1x03_P2.50mm_Vertical -> GS_Connectors:JST_XH_S3B-XH-A-1_1x03_P2.50mm_Horizontal
- JP1: value SW.SIG_INVERSION -> SW_INVERSION; moved to B.Cu
- S1, SW1, TP1, TP2, TP3, TP4, TP5, TP6: moved to B.Cu
- moved R4 151.0 mm to (240.8, 113.0), turned to 90 degrees
- moved TP1 135.3 mm to (248.9, 97.8), turned to 180 degrees
- moved TP2 135.2 mm to (248.9, 102.9), turned to 180 degrees
- moved C4 134.7 mm to (242.6, 87.7), turned to -90 degrees
- moved U1 133.6 mm to (226.1, 101.6), turned to 90 degrees
- moved H2 131.7 mm to (247.7, 88.9)
- moved C6 129.9 mm to (237.5, 103.5), turned to 90 degrees
- moved R5 129.9 mm to (221.6, 101.0), turned to -90 degrees
- moved R2 129.6 mm to (216.5, 113.7), turned to 90 degrees
- moved TP6 128.2 mm to (248.9, 100.3), turned to 180 degrees
- moved C2 125.9 mm to (233.7, 88.3)
- moved R6 125.4 mm to (217.2, 88.3)
- moved S1 123.8 mm to (246.4, 109.2), turned to 180 degrees
- moved R1 116.7 mm to (206.4, 96.5)
- moved TP5 116.7 mm to (237.5, 108.0), turned to 180 degrees
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Connections:
- J1 pad 2: +3.3V -> /SIG.OUT
- J1 pad 3: /SIG.OUT -> +3.3V
- R2 pad 1: Net-(U1-+) -> Net-(U2A-+)
- R5 pad 2: Net-(U1-+) -> Net-(U2A-+)
Routing:
- net +3.3V: track 0.00 -> 117.6 mm
- net /SIG.OUT: track 0.00 -> 53.3 mm
- net Net-(J2-Pin_1): track 0.00 -> 41.8 mm
- net Net-(U1-+): track 0.00 -> 25.0 mm
- net Net-(U1--): track 0.00 -> 24.0 mm
- net Net-(J2-Pin_2): track 0.00 -> 21.0 mm
- net Net-(U2A-+): track 0.00 -> 16.2 mm
- net Net-(JP1-B): track 0.00 -> 14.0 mm
- net Net-(C4-Pad1): track 0.00 -> 3.85 mm
- net Net-(C3-Pad1): track 0.00 -> 3.81 mm
- net GND: track 0.00 -> 3.79 mm, vias 0 -> 37
- added copper zone on B.Cu, net GND
- added copper zone on F.Cu, net GND
Other:
- board outline added: 58.4 x 31.8 mm
- board text added: "0"
- board text added: "0 mm"
- board text added: "0.01 mm"
- board text added: "0.02"
- board text added: "0.035 mm"
- board text added: "0.1000 mm / 0.1000 mm"
- board text added: "0.3000 mm"
- board text added: "1"
- board text added: "1.51 mm"
- board text added: "1.6000 mm"
- board text added: "10ms time constant 1V of hysteresis"
- board text added: "2"
- board text added: "3.3"
- board text added: "3V3"
- board text added: "4.5"
- board text added: "58.4200 mm x 31.7500 mm"
- board text added: "B.Cu"
- board text added: "B.Mask"
- board text added: "B.Paste"
- board text added: "B.Silkscreen"
- board text added: "BOARD CHARACTERISTICS"
- board text added: "Board Thickness:"
- board text added: "Board overall dimensions:"
- board text added: "Bottom Silk Screen"
- board text added: "Bottom Solder Mask"
- board text added: "Bottom Solder Paste"
- board text added: "C"
- board text added: "Castellated pads:"
- board text added: "Color"
- board text added: "Copper Finish:"
- board text added: "Copper Layer Count:"
- board text added: "Designed by George Sleen"
- board text added: "Dielectric 1"
- board text added: "Edge card connectors:"
- board text added: "Epsilon R"
- board text added: "F.Cu"
- board text added: "F.Mask"
- board text added: "F.Paste"
- board text added: "F.Silkscreen"
- board text added: "FR4"
- board text added: "GND"
- board text added: "Impedance Control:"
- board text added: "Layer Name"
- board text added: "Loss Tangent"
- board text added: "Material"
- board text added: "Min hole diameter:"
- board text added: "Min track/spacing:"
- board text added: "NC"
- board text added: "NO"
- board text added: "No"
- board text added: "None"
- board text added: "Not specified"
- board text added: "OUT"
- board text added: "Plated Board Edge:"
- board text added: "RC Debouncer"
- board text added: "RC Network"
- board text added: "Thickness (mm)"
- board text added: "Top Silk Screen"
- board text added: "Top Solder Mask"
- board text added: "Top Solder Paste"
- board text added: "Type"
- board text added: "copper"
- board text added: "core"
- board text added: "github.com /enph253-2025-team5 /rc-debouncing-pcb"

Commit message: Update back silkscreen to include revision
Other:
- board text added: "${REVISION}"
