File: rc-debouncer/rc-debouncer.kicad_sch (KiCad schematic)
At the start: 0 parts

Commit message: Layout first revision
Parts:
- added C1, C2, C6: 100nF, Capacitor_THT:C_Disc_D3.0mm_W2.0mm_P2.50mm, symbol GS_Capacitor_THT:C_THT_Ceramic_Disk
- added C3, C4: 100nF, Capacitor_THT:C_Disc_D3.0mm_W2.0mm_P2.50mm, symbol GS_Capacitor_THT:C_THT_100nF
- added C5: 10uF, Capacitor_THT:CP_Radial_D5.0mm_P2.00mm, symbol GS_Capacitor_THT:C_THT_Electrolytic_Radial
- added H1, H2: M3_PTH, MountingHole:MountingHole_3.2mm_M3_Pad, symbol Mechanical:MountingHole_Pad
- added J1: MCU, Connector_JST:JST_XH_B3B-XH-A_1x03_P2.50mm_Vertical, symbol Connector:Conn_01x03_Socket
- added J2: SIG.IN, TerminalBlock:TerminalBlock_Xinya_XY308-2.54-2P_1x02_P2.54mm_Horizontal, symbol GS_Connectors:Screw_Terminal_01x02_2.54mm_Xinya
- added JP1: SW.SIG_INVERSION, Jumper:SolderJumper-3_P1.3mm_Bridged12_RoundedPad1.0x1.5mm, symbol Jumper:SolderJumper_3_Bridged12
- added R1, R2, R5, R6: 100k, Resistor_THT:R_Axial_DIN0309_L9.0mm_D3.2mm_P12.70mm_Horizontal, symbol GS_Resistor_THT:R_250mW
- added R3, R4: 1k, Resistor_THT:R_Axial_DIN0309_L9.0mm_D3.2mm_P12.70mm_Horizontal, symbol GS_Resistor_THT:R_250mW
- added S1: Logo, GS_Virtual:ENPH253_Logo, symbol GS_Virtual:ENPH253_Logo
- added SW1: Input, Button_Switch_THT:SW_XKB_DM1-16UP-1, symbol GS_Switches:SW_SPDT_XKB_WK1-X-TIAIHUA
- added TP1: 3.3V, TestPoint:TestPoint_Pad_1.5x1.5mm, symbol Connector:TestPoint_Small
- added TP2: GND, TestPoint:TestPoint_Pad_1.5x1.5mm, symbol Connector:TestPoint_Small
- added TP3: SIG.RC_FILTERED, TestPoint:TestPoint_Pad_1.5x1.5mm, symbol Connector:TestPoint_Small
- added TP4: SIG.RAW, TestPoint:TestPoint_Pad_1.5x1.5mm, symbol Connector:TestPoint_Small
- added TP5: V_REF, TestPoint:TestPoint_Pad_1.5x1.5mm, symbol Connector:TestPoint_Small
- added TP6: SIG.OUT, TestPoint:TestPoint_Pad_1.5x1.5mm, symbol Connector:TestPoint_Small
- added U1: LM311, Package_DIP:DIP-8_W7.62mm_LongPads, symbol GS_Comparators:LM311
Connections:
- new net: J2.1 (Pin_1), R3.2, R6.1, SW1.1 (C), TP4.1
- new net: C3.1, H1.1
- new net: C2.1, R6.2, TP3.1, U1.3 (-)
- new net: R1.2, R2.1, R5.2, TP5.1, U1.2 (+)
- new net: J2.2 (Pin_2), JP1.1 (A), SW1.2 (NO)
- new net: JP1.3 (B), SW1.3 (NC)
- new net: C4.1, H2.1
- new net +3.3V: C1.1, C5.1, C6.1, J1.2 (Pin_2), R2.2, R3.1, R4.1, TP1.1, U1.8 (V+)
- new net GND: C1.2, C2.2, C3.2, C4.2, C5.2, C6.2, J1.1 (Pin_1), JP1.2 (C), R5.1, TP2.1, U1.1 (EMIT), U1.4 (V-)
- new net SIG.OUT: J1.3 (Pin_3), R1.1, R4.2, TP6.1, U1.7
- no-connect marks 0 -> 2

Commit message: Finish layout and generate production outputs
Parts:
- added C7: 100nF, Capacitor_THT:C_Disc_D3.0mm_W2.0mm_P2.50mm, symbol GS_Capacitor_THT:C_THT_Ceramic_Disk
- added U2: LM358, Package_DIP:DIP-8_W7.62mm_LongPads, symbol Amplifier_Operational:LM358
- J1: footprint Connector_JST:JST_XH_B3B-XH-A_1x03_P2.50mm_Vertical -> GS_Connectors:JST_XH_S3B-XH-A-1_1x03_P2.50mm_Horizontal
- JP1: value SW.SIG_INVERSION -> SW_INVERSION
Connections:
- net +3.3V: now also J1.3 (Pin_3), C7.1, U2.8 (V+); no longer J1.2 (Pin_2)
- net GND: now also C7.2, U2.4 (V-)
- net SIG.OUT: now also J1.2 (Pin_2); no longer J1.3 (Pin_3)
- net at R1.2, TP5.1, U1.2 (+): now also U2.1, U2.2 (-); no longer R2.1, R5.2
- new net: R2.1, R5.2, U2.3 (+)
- no-connect marks 2 -> 5
Other:
- moved on the sheet: C1, C2, J2, JP1, R1, R2, R3, R4, R5, R6, SW1, TP3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
